File: Documents/Pcb/client/wssf_arduino_nano_client.brd (EAGLE design)
At the start: 54 x 38 mm, 12 parts

Commit message: update pcbs and add gerbers files
Parts:
- moved C1 1.00 mm to (12.6, 28.9)
Routing:
- net GND: track 82.0 -> 81.0 mm, vias 0 -> 6
- added copper zone on layer 1, net GND
- added copper zone on layer 16, net GND
Other:
- board text added: "+"
- board text added: "WSFF Client v1.0 Assouline Yohann 21/12/2020"
- board text added: "btn1"
- board text added: "btn2"
- board text added: "captouch"
Changed lines of the file:
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@@
 <setting verticaltext="up"/>
 </settings>
-<grid distance="50" unitdist="mil" unit="mil" style="lines" multiple="1" display="no" altdistance="5" altunitdist="mil" altunit="mil"/>
+<grid distance="1" unitdist="mm" unit="mm" style="lines" multiple="1" display="yes" altdistance="1" altunitdist="mm" altunit="mm"/>
 <layers>
 <layer number="1" name="Top" color="4" fill="1" visible="yes" active="yes"/>
@@
 </layers>
 <board>
-<fusionsync huburn="a.YnVzaW5lc3M6ZXBpdGVjaDQw" projecturn="a.YnVzaW5lc3M6ZXBpdGVjaDQwI0QyMDIwMDMxMDI3MzUwNDYwMQ" f3durn="urn:adsk.wipprod:dm.lineage:smIWb7I_QH2r5atMStTLYg" pcbguid="" lastpulledtime="" lastsyncedchangeguid="" latestrevisionid="9e3c73c2-d581-4510-a2eb-30fbacaf7552" lastsyncedrevisionid="9e3c73c2-d581-4510-a2eb-30fbacaf7552" lastboardhashguid="ab5e6a2c-8e40-022e-9127-97815b74cb21" lastpushedtime="2020-12-15T17:08:11Z" linktopcb3d="true"/>
+<fusionsync huburn="a.YnVzaW5lc3M6ZXBpdGVjaDQw" projecturn="a.YnVzaW5lc3M6ZXBpdGVjaDQwI0QyMDIwMDMxMDI3MzUwNDYwMQ" f3durn="urn:adsk.wipprod:dm.lineage:smIWb7I_QH2r5atMStTLYg" pcbguid="" lastpulledtime="" lastsyncedchangeguid="" latestrevisionid="8f84e580-4472-4ef0-a48f-53cddb32db01" lastsyncedrevisionid="8f84e580-4472-4ef0-a48f-53cddb32db01" lastboardhashguid="d33897f3-c5e7-9f18-0b40-dca484aeffb9" lastpushedtime="2020-12-21T22:48:16Z" linktopcb3d="true"/>
 <plain>
-<hole x="52.72" y="36.56" drill="1.397"/>
-<hole x="1.27" y="1.08" drill="1.397"/>
-<hole x="1.27" y="36.56" drill="1.397"/>
-<hole x="52.72" y="1.08" drill="1.397"/>
+<hole x="52" y="36" drill="1.5"/>
+<hole x="2" y="2" drill="1.5"/>
+<hole x="2" y="36" drill="1.5"/>
+<hole x="52" y="2" drill="1.5"/>
 <wire x1="0" y1="0" x2="0" y2="38" width="0.1524" layer="20"/>
 <wire x1="0" y1="38" x2="54" y2="38" width="0.1524" layer="20"/>
@@
 <dimension x1="54" y1="0" x2="0" y2="0" x3="27" y3="-3" textsize="1.778" layer="20"/>
 <dimension x1="0" y1="0" x2="0" y2="38" x3="-2" y3="19" textsize="1.778" layer="20"/>
+<text x="7" y="2" size="0.5" layer="21">captouch</text>
+<text x="34" y="2" size="0.5" layer="21">btn2</text>
+<text x="48" y="4" size="0.5" layer="21">btn1</text>
+<text x="16" y="2" size="0.5" layer="21">+</text>
+<text x="52" y="5" size="0.5" layer="21" rot="R90">WSFF Client v1.0
+Assouline Yohann
+21/12/2020</text>
 </plain>
 <attributes>
@@
 </element>
 <element name="GND" library="pinhead" library_urn="urn:adsk.eagle:library:325" package="1X01" package3d_urn="urn:adsk.eagle:package:22485/2" value="" x="4.81" y="35.29" smashed="yes">
-<attribute name="NAME" x="3.9238" y="32.0388" size="1.27" layer="25" ratio="10"/>
+<attribute name="NAME" x="3.9238" y="33.0388" size="0.5" layer="25" ratio="10"/>
 <attribute name="POPULARITY" value="64" x="32.75" y="13.7" size="1.778" layer="27" display="off"/>
 <attribute name="VALUE" x="3.54" y="32.115" size="1.27" layer="27"/>
 </element>
 <element name="VCC" library="pinhead" library_urn="urn:adsk.eagle:library:325" package="1X01" package3d_urn="urn:adsk.eagle:package:22485/2" value="" x="9.18" y="35.29" smashed="yes">
-<attribute name="NAME" x="9.5638" y="32.0388" size="1.27" layer="25" ratio="10"/>
+<attribute name="NAME" x="8.5638" y="33.0388" size="0.5" layer="25" ratio="10"/>
 <attribute name="POPULARITY" value="64" x="42.2" y="13.7" size="1.778" layer="27" display="off"/>
 <attribute name="VALUE" x="7.91" y="32.115" size="1.27" layer="27"/>
 </element>
 <element name="NRF24L01" library="diy-modules" package="WIRELESS-NRF24L01" value="WIRELESS-NRF24L01" x="34.86" y="29.02" smashed="yes">
-<attribute name="NAME" x="34.86" y="34.1" size="1.27" layer="25" align="bottom-center"/>
+<attribute name="NAME" x="34.86" y="32.1" size="1.27" layer="25" align="bottom-center"/>
 </element>
 <element name="LED1" library="led" library_urn="urn:adsk.eagle:library:259" package="LED5MM" package3d_urn="urn:adsk.eagle:package:15799/2" value="" x="18.97" y="2.08" smashed="yes">
@@
 <attribute name="VALUE" x="22.1704" y="0.2766" size="1.27" layer="27" ratio="10"/>
 </element>
-<element name="C1" library="rcl" library_urn="urn:adsk.eagle:library:334" package="E2-5" package3d_urn="urn:adsk.eagle:package:23346/2" value="10uF" x="12.64" y="27.94" smashed="yes" rot="R180">
-<attribute name="POPULARITY" value="7" x="12.64" y="27.94" size="1.778" layer="27" rot="R180" display="off"/>
-<attribute name="SPICEPREFIX" value="C" x="12.64" y="27.94" size="1.778" layer="27" rot="R180" display="off"/>
+<element name="C1" library="rcl" library_urn="urn:adsk.eagle:library:334" package="E2-5" package3d_urn="urn:adsk.eagle:package:23346/2" value="10uF" x="12.64" y="28.94" smashed="yes" rot="R180">
+<attribute name="POPULARITY" value="7" x="12.64" y="28.94" size="1.778" layer="27" rot="R180" display="off"/>
+<attribute name="SPICEPREFIX" value="C" x="12.64" y="28.94" size="1.778" layer="27" rot="R180" display="off"/>
 </element>
 <element name="CON_CAPTOUCH" library="SparkFun-Connectors" library_urn="urn:adsk.eagle:library:513" package="1X01" package3d_urn="urn:adsk.eagle:package:38028/1" value="" x="5.08" y="2.08" smashed="yes">
@@
 <attribute name="POPULARITY" value="48" x="47.48" y="13.24" size="1.778" layer="27" rot="R270" display="off"/>
 <attribute name="SPICEPREFIX" value="R" x="47.48" y="13.24" size="1.778" layer="27" rot="R270" display="off"/>
-<attribute name="VALUE" x="46.9974" y="13.8656" size="0.9906" layer="27" ratio="10" rot="R270"/>
+<attribute name="VALUE" x="46.9974" y="13.8656" size="0.9906" layer="21" ratio="10" rot="R270"/>
 </element>
 <element name="R2" library="rcl" library_urn="urn:adsk.eagle:library:334" package="0204/7" package3d_urn="urn:adsk.eagle:package:23498/2" value="1M" x="2.67" y="27.24" smashed="yes" rot="R90">
 <attribute name="POPULARITY" value="48" x="2.67" y="27.24" size="1.778" layer="27" rot="R90" display="off"/>
 <attribute name="SPICEPREFIX" value="R" x="2.67" y="27.24" size="1.778" layer="27" rot="R90" display="off"/>
-<attribute name="VALUE" x="3.1526" y="26.6144" size="0.9906" layer="27" ratio="10" rot="R90"/>
+<attribute name="VALUE" x="3.1526" y="26.6144" size="0.9906" layer="21" ratio="10" rot="R90"/>
 </element>
 <element name="R1" library="rcl" library_urn="urn:adsk.eagle:library:334" package="0204/7" package3d_urn="urn:adsk.eagle:package:23498/2" value="1M" x="5.86" y="27.24" smashed="yes" rot="R90">
 <attribute name="POPULARITY" value="48" x="5.86" y="27.24" size="1.778" layer="27" rot="R90" display="off"/>
 <attribute name="SPICEPREFIX" value="R" x="5.86" y="27.24" size="1.778" layer="27" rot="R90" display="off"/>
-<attribute name="VALUE" x="6.3426" y="26.6144" size="0.9906" layer="27" ratio="10" rot="R90"/>
+<attribute name="VALUE" x="6.3426" y="26.6144" size="0.9906" layer="21" ratio="10" rot="R90"/>
 </element>
 </elements>
@@
 <contactref element="ARDUINO_NANO1" pad="14"/>
 <wire x1="11.5" y1="32.25" x2="11.5" y2="31" width="0.2" layer="1"/>
-<wire x1="11.5" y1="31" x2="11.5" y2="28" width="0.2" layer="1"/>
-<wire x1="11.5" y1="28" x2="11.624" y2="27.94" width="0.2" layer="1"/>
+<wire x1="11.5" y1="31" x2="11.5" y2="29" width="0.2" layer="1"/>
+<wire x1="11.5" y1="29" x2="11.624" y2="28.94" width="0.2" layer="1"/>
 <wire x1="11.5" y1="32.25" x2="6.87666875" y2="33.22333125" width="0.2" layer="1"/>
 <wire x1="6.87666875" y1="33.22333125" x2="4.81" y2="35.29" width="0.2" layer="1"/>
@@
 <wire x1="22.25" y1="35.25" x2="22.16" y2="35.37" width="0.2" layer="1"/>
 <wire x1="33.25" y1="20" x2="33.29" y2="19.86" width="0.2" layer="1"/>
+<polygon width="0.1524" layer="16" isolate="0.4064">
+<vertex x="0" y="0"/>
+<vertex x="0" y="38"/>
+<vertex x="54" y="38"/>
+<vertex x="54" y="0"/>
+</polygon>
+<via x="10" y="13" extent="1-16" drill="0.35"/>
+<via x="32" y="10" extent="1-16" drill="0.35"/>
+<via x="50" y="19" extent="1-16" drill="0.35"/>
+<via x="39" y="29" extent="1-16" drill="0.35"/>
+<via x="19" y="13" extent="1-16" drill="0.35"/>
+<via x="15" y="33" extent="1-16" drill="0.35"/>
+<polygon width="0.1524" layer="1" isolate="0.4064">
+<vertex x="0" y="0"/>
+<vertex x="0" y="38"/>
+<vertex x="54" y="38"/>
+<vertex x="54" y="0"/>
+</polygon>
 </signal>
 <signal name="5V">
@@
 <wire x1="12" y1="20" x2="8" y2="16" width="0.2" layer="16"/>
 <wire x1="12" y1="26.25" x2="12" y2="20" width="0.2" layer="16"/>
-<wire x1="13.5" y1="27.75" x2="12" y2="26.25" width="0.2" layer="16"/>
 <wire x1="8" y1="4.75" x2="7.89" y2="4.62" width="0.2" layer="16"/>
-<wire x1="13.5" y1="27.75" x2="13.656" y2="27.94" width="0.2" layer="16"/>
+<wire x1="13.656" y1="28.94" x2="13.656" y2="28.266921875" width="0.2" layer="16"/>
+<wire x1="13.656" y1="28.266921875" x2="12" y2="26.25" width="0.2" layer="16"/>
 <wire x1="24" y1="35.25" x2="24.5" y2="35.25" width="0.2" layer="16"/>
 <wire x1="22.75" y1="34" x2="24" y2="35.25" width="0.2" layer="16"/>
 <wire x1="19.75" y1="34" x2="22.75" y2="34" width="0.2" layer="16"/>
-<wire x1="13.75" y1="28" x2="19.75" y2="34" width="0.2" layer="16"/>
+<wire x1="16.51470625" y1="30.76470625" x2="19.75" y2="34" width="0.2" layer="16"/>
 <wire x1="24.5" y1="35.25" x2="24.7" y2="35.37" width="0.2" layer="16"/>
-<wire x1="13.75" y1="28" x2="13.656" y2="27.94" width="0.2" layer="16"/>
+<wire x1="16.51470625" y1="30.76470625" x2="13.656" y2="28.94" width="0.2" layer="16"/>
 </signal>
 </signals>
@@
 </drawing>
 <compatibility>
+<note version="6.3" minversion="6.2.2" severity="warning">
+Since Version 6.2.2 text objects can contain more than one line,
+which will not be processed correctly with this version.
+</note>
 <note version="8.2" severity="warning">
 Since Version 8.2, EAGLE supports online libraries. The ids
