File: Documents/Pcb/server/wssf_arduino_nano_server.sch (EAGLE design)
At the start: 10 parts

Commit message: update pcbs and add gerbers files
Changed lines of the file:
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@@
 </instance>
 <instance part="NP_VCC" gate="G$1" x="-5.08" y="76.2" smashed="yes">
-<attribute name="NAME" x="-16.51" y="84.455" size="1.778" layer="95"/>
+<attribute name="NAME" x="-11.43" y="79.375" size="1.778" layer="95"/>
 <attribute name="VALUE" x="-11.43" y="71.12" size="1.778" layer="96"/>
 </instance>
 <instance part="NP_GND" gate="G$1" x="-5.08" y="58.42" smashed="yes">
-<attribute name="NAME" x="-19.05" y="64.135" size="1.778" layer="95"/>
+<attribute name="NAME" x="-11.43" y="61.595" size="1.778" layer="95"/>
 <attribute name="VALUE" x="-11.43" y="53.34" size="1.778" layer="96"/>
 </instance>
