File: Documents/PCB/client/wssf_client.brd (EAGLE design)
At the start: 54 x 38 mm, 16 parts, among them M1 ARDUINO-NANO-3.0, M2 WIRELESS-NRF24L01

Commit message: update PCBS and add screenshots
Parts:
- R4: value X -> ?
Changed lines of the file:
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@@
 <drawing>
 <settings>
-<setting alwaysvectorfont="no"/>
+<setting alwaysvectorfont="yes"/>
 <setting verticaltext="up"/>
 </settings>
@@
 <attribute name="POPULARITY" value="48" x="8.5" y="28" size="1.778" layer="27" rot="R270" display="off"/>
 <attribute name="SPICEPREFIX" value="R" x="8.5" y="28" size="1.778" layer="27" rot="R270" display="off"/>
-<attribute name="VALUE" x="8.0174" y="29.6256" size="0.9906" layer="27" ratio="10" rot="R270"/>
+<attribute name="VALUE" x="8.0174" y="29.6256" size="0.9906" layer="25" ratio="10" rot="R270"/>
 </element>
 <element name="R2" library="rcl" library_urn="urn:adsk.eagle:library:334" package="0204/7" package3d_urn="urn:adsk.eagle:package:23498/2" value="1M" x="2.5" y="28" smashed="yes" rot="R270">
 <attribute name="POPULARITY" value="48" x="2.5" y="28" size="1.778" layer="27" rot="R270" display="off"/>
 <attribute name="SPICEPREFIX" value="R" x="2.5" y="28" size="1.778" layer="27" rot="R270" display="off"/>
-<attribute name="VALUE" x="2.0174" y="29.6256" size="0.9906" layer="27" ratio="10" rot="R270"/>
+<attribute name="VALUE" x="2.0174" y="29.6256" size="0.9906" layer="25" ratio="10" rot="R270"/>
 </element>
 <element name="R3" library="rcl" library_urn="urn:adsk.eagle:library:334" package="0204/7" package3d_urn="urn:adsk.eagle:package:23498/2" value="10k" x="48" y="17" smashed="yes" rot="R180">
 <attribute name="POPULARITY" value="48" x="48" y="17" size="1.778" layer="27" rot="R180" display="off"/>
 <attribute name="SPICEPREFIX" value="R" x="48" y="17" size="1.778" layer="27" rot="R180" display="off"/>
-<attribute name="VALUE" x="49.6256" y="17.4826" size="0.9906" layer="27" ratio="10" rot="R180"/>
+<attribute name="VALUE" x="49.6256" y="17.4826" size="0.9906" layer="25" ratio="10" rot="R180"/>
 </element>
 <element name="D1" library="SparkFun-LED" library_urn="urn:adsk.eagle:library:529" package="LED-RGB-THRU" package3d_urn="urn:adsk.eagle:package:39368/1" value="CLEAR" x="19.5" y="2.5" smashed="yes">
@@
 <attribute name="POPULARITY" value="48" x="50.5" y="9" size="1.778" layer="27" rot="R270" display="off"/>
 <attribute name="SPICEPREFIX" value="R" x="50.5" y="9" size="1.778" layer="27" rot="R270" display="off"/>
-<attribute name="VALUE" x="50.0174" y="10.6256" size="0.9906" layer="27" ratio="10" rot="R270"/>
+<attribute name="VALUE" x="50.0174" y="10.6256" size="0.9906" layer="25" ratio="10" rot="R270"/>
 </element>
 <element name="R_LED2" library="rcl" library_urn="urn:adsk.eagle:library:334" package="0204/7" package3d_urn="urn:adsk.eagle:package:23498/2" value="220" x="48" y="9" smashed="yes" rot="R270">
 <attribute name="POPULARITY" value="48" x="48" y="9" size="1.778" layer="27" rot="R270" display="off"/>
 <attribute name="SPICEPREFIX" value="R" x="48" y="9" size="1.778" layer="27" rot="R270" display="off"/>
-<attribute name="VALUE" x="47.5174" y="10.6256" size="0.9906" layer="27" ratio="10" rot="R270"/>
+<attribute name="VALUE" x="47.5174" y="10.6256" size="0.9906" layer="25" ratio="10" rot="R270"/>
 </element>
 <element name="R_LED3" library="rcl" library_urn="urn:adsk.eagle:library:334" package="0204/7" package3d_urn="urn:adsk.eagle:package:23498/2" value="220" x="45.5" y="9" smashed="yes" rot="R270">
 <attribute name="POPULARITY" value="48" x="45.5" y="9" size="1.778" layer="27" rot="R270" display="off"/>
 <attribute name="SPICEPREFIX" value="R" x="45.5" y="9" size="1.778" layer="27" rot="R270" display="off"/>
-<attribute name="VALUE" x="45.0174" y="10.6256" size="0.9906" layer="27" ratio="10" rot="R270"/>
-</element>
-<element name="R4" library="rcl" library_urn="urn:adsk.eagle:library:334" package="0204/7" package3d_urn="urn:adsk.eagle:package:23498/2" value="X" x="5.5" y="28" smashed="yes" rot="R270">
+<attribute name="VALUE" x="45.0174" y="10.6256" size="0.9906" layer="25" ratio="10" rot="R270"/>
+</element>
+<element name="R4" library="rcl" library_urn="urn:adsk.eagle:library:334" package="0204/7" package3d_urn="urn:adsk.eagle:package:23498/2" value="?" x="5.5" y="28" smashed="yes" rot="R270">
 <attribute name="NAME" x="6.7954" y="30.54" size="0.9906" layer="25" ratio="10" rot="R270"/>
 <attribute name="POPULARITY" value="48" x="5.5" y="28" size="1.778" layer="27" rot="R270" display="off"/>
 <attribute name="SPICEPREFIX" value="R" x="5.5" y="28" size="1.778" layer="27" rot="R270" display="off"/>
-<attribute name="VALUE" x="5.0174" y="29.6256" size="0.9906" layer="27" ratio="10" rot="R270"/>
+<attribute name="VALUE" x="5.0174" y="29.6256" size="0.9906" layer="25" ratio="10" rot="R270"/>
 </element>
 </elements>
