File: Documents/PCB/client/wssf_client.sch (EAGLE design)
At the start: 16 parts, among them M1 ARDUINO-NANO-3.0, M2 WIRELESS-NRF24L01

Commit message: update PCBS and add screenshots
Parts:
- R4: value X -> ?
Changed lines of the file:
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@@
 <part name="R_LED3" library="rcl" library_urn="urn:adsk.eagle:library:334" deviceset="R-US_" device="0204/7" package3d_urn="urn:adsk.eagle:package:23498/2" value="220"/>
 <part name="GND2" library="supply1" library_urn="urn:adsk.eagle:library:371" deviceset="GND" device=""/>
-<part name="R4" library="rcl" library_urn="urn:adsk.eagle:library:334" deviceset="R-US_" device="0204/7" package3d_urn="urn:adsk.eagle:package:23498/2" value="X"/>
+<part name="R4" library="rcl" library_urn="urn:adsk.eagle:library:334" deviceset="R-US_" device="0204/7" package3d_urn="urn:adsk.eagle:package:23498/2" value="?"/>
 </parts>
 <sheets>
