File: Documents/PCB/server/wssf_server.brd (EAGLE design)
At the start: 44 x 52 mm, 14 parts, among them M1 ARDUINO-NANO-3.0, M2 WIRELESS-NRF24L01

Commit message: update PCBS and add screenshots
Changed lines of the file:
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@@
 <drawing>
 <settings>
-<setting alwaysvectorfont="no"/>
+<setting alwaysvectorfont="yes"/>
 <setting verticaltext="up"/>
 </settings>
@@
 <element name="BZR_GND" library="pinhead" library_urn="urn:adsk.eagle:library:325" package="1X01" package3d_urn="urn:adsk.eagle:package:22485/2" value="BZR_GND" x="21" y="50" smashed="yes">
 <attribute name="POPULARITY" value="64" x="21" y="50" size="1.778" layer="27" display="off"/>
-<attribute name="VALUE" x="19.73" y="47.825" size="0.7" layer="27"/>
+<attribute name="VALUE" x="19.73" y="47.825" size="0.7" layer="25"/>
 </element>
 <element name="BZR_VCC" library="pinhead" library_urn="urn:adsk.eagle:library:325" package="1X01" package3d_urn="urn:adsk.eagle:package:22485/2" value="BZR_VCC" x="26" y="50" smashed="yes">
 <attribute name="POPULARITY" value="64" x="26" y="50" size="1.778" layer="27" display="off"/>
-<attribute name="VALUE" x="24.73" y="47.825" size="0.7" layer="27"/>
+<attribute name="VALUE" x="24.73" y="47.825" size="0.7" layer="25"/>
 </element>
 <element name="M1" library="wsff_lib" package="ARDUINO-NANO-3.0" value="ARDUINO-NANO-3.0" x="32" y="26" smashed="yes" rot="R90"/>
