File: Documents/PCB/server/touche_server.brd (EAGLE design)
At the start: 44 x 52 mm, 14 parts, among them M1 ARDUINO-NANO-3.0, M2 WIRELESS-NRF24L01

Commit message: update pcb
Parts:
- renumbered BTN_PISTE_MODE to BTN_SWITCH, CHANGE_WEAPON to BTN_PISTE, SWITCH_PLAYERS to BTN_CHANGE_WP
Connections:
- removed net N$1: BZR_GND.1, POT_5K.3
- removed net PIN_BTN_SWITCH_PLAYERS: BTN_CHANGE_WP.1, M1.J1.9
- new net PIN_BTN_SWITCH_SIDE: BTN_SWITCH.1, M1.J1.7
- new net POT_IN: M1.J2.9, POT_5K.2
- net GND: now also BZR_GND.1, POT_5K.1; no longer POT_5K.2
- net PIN_BTN_CHANGE_WEAPON: now also BTN_CHANGE_WP.1, M1.J1.9; no longer BTN_PISTE.1, M1.J1.8
- net PIN_BTN_PISTE_MODE: now also BTN_PISTE.1, M1.J1.8; no longer BTN_SWITCH.1, M1.J1.7
- net VCC: now also POT_5K.3
Routing:
- net POT_IN: track 0.00 -> 35.5 mm
- net PIN_BTN_SWITCH_SIDE: track 0.00 -> 31.7 mm
- net PIN_BTN_SWITCH_PLAYERS: track 22.2 -> 0.00 mm
- net VCC: track 75.5 -> 92.3 mm
- net N$1: track 15.3 -> 0.00 mm
- net PIN_BTN_PISTE_MODE: track 31.7 -> 25.3 mm
- net PIN_BTN_CHANGE_WEAPON: track 25.3 -> 22.2 mm
Other:
- outline, holes or cut-outs redrawn
- board text added: "Touche Server v1.0 Assouline Yohann 07/09/2021"
- board text removed: "WSFF Server v1.0 Assouline Yohann 11/04/2021"
Changed lines of the file:
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@@
 <drawing>
 <settings>
-<setting alwaysvectorfont="yes"/>
+<setting alwaysvectorfont="no"/>
 <setting verticaltext="up"/>
 </settings>
@@
 </layers>
 <board>
-<fusionsync huburn="a.YnVzaW5lc3M6ZXBpdGVjaDQw" projecturn="a.YnVzaW5lc3M6ZXBpdGVjaDQwI0QyMDIwMDMxMDI3MzUwNDYwMQ" f3durn="urn:adsk.wipprod:dm.lineage:Yh6YGJO4SySBV2_jDXAEDA" pcbguid="" lastpulledtime="" lastsyncedchangeguid="" latestrevisionid="a7b8685e-58eb-4f31-9868-9bd4014e3094" lastsyncedrevisionid="a7b8685e-58eb-4f31-9868-9bd4014e3094" lastboardhashguid="a583c829-d65a-f32f-4a9e-8cbcd4971de8" lastpushedtime="2021-04-10T23:12:16Z" linktopcb3d="true"/>
+<fusionsync huburn="a.YnVzaW5lc3M6ZXBpdGVjaDQw" projecturn="a.YnVzaW5lc3M6ZXBpdGVjaDQwI0QyMDIwMDMxMDI3MzUwNDYwMQ" f3durn="urn:adsk.wipprod:dm.lineage:Yh6YGJO4SySBV2_jDXAEDA" pcbguid="" lastpulledtime="" lastsyncedchangeguid="" latestrevisionid="79447381-6fe7-4767-a0dc-130f9d462c66" lastsyncedrevisionid="79447381-6fe7-4767-a0dc-130f9d462c66" lastboardhashguid="3b59297b-7802-3bfe-cc7e-d27ae015b3fb" lastpushedtime="2021-06-07T21:33:41Z" linktopcb3d="true"/>
 <plain>
-<hole x="42" y="50" drill="1.397"/>
-<hole x="2" y="2" drill="1.397"/>
-<hole x="2" y="50" drill="1.5"/>
-<hole x="42" y="2" drill="1.397"/>
-<wire x1="0" y1="0" x2="0" y2="52" width="0.1524" layer="20"/>
-<wire x1="0" y1="52" x2="44" y2="52" width="0.1524" layer="20"/>
-<wire x1="44" y1="52" x2="44" y2="0" width="0.1524" layer="20"/>
-<wire x1="44" y1="0" x2="0" y2="0" width="0.1524" layer="20"/>
+<hole x="42" y="50" drill="1.8"/>
+<hole x="2" y="2" drill="1.8"/>
+<hole x="2" y="50" drill="1.8"/>
+<hole x="42" y="2" drill="1.8"/>
+<wire x1="42" y1="0" x2="2" y2="0" width="0.1524" layer="20"/>
+<wire x1="2" y1="0" x2="0" y2="2" width="0.1524" layer="20" curve="-90"/>
+<wire x1="0" y1="2" x2="0" y2="50" width="0.1524" layer="20"/>
+<wire x1="0" y1="50" x2="2" y2="52" width="0.1524" layer="20" curve="-90"/>
+<wire x1="2" y1="52" x2="42" y2="52" width="0.1524" layer="20"/>
+<wire x1="42" y1="52" x2="44" y2="50" width="0.1524" layer="20" curve="-90"/>
+<wire x1="44" y1="50" x2="44" y2="2" width="0.1524" layer="20"/>
+<wire x1="44" y1="2" x2="42" y2="0" width="0.1524" layer="20" curve="-90"/>
 <dimension x1="44" y1="0" x2="0" y2="0" x3="22" y3="-3" textsize="1.778" layer="20"/>
 <dimension x1="0" y1="0" x2="0" y2="52" x3="-5" y3="26" textsize="1.778" layer="20"/>
-<text x="37" y="30" size="1.2" layer="21" rot="SR270" align="top-right">WSFF Server v1.0
+<text x="37" y="30" size="1.2" layer="21" rot="SR270" align="top-right">Touche Server v1.0
 Assouline Yohann
-11/04/2021</text>
+07/09/2021</text>
 </plain>
 <attributes>
@@
 <attribute name="VALUE" x="15.54" y="46.175" size="1.27" layer="27" rot="R270"/>
 </element>
-<element name="BTN_PISTE_MODE" library="SparkFun-Switches" library_urn="urn:adsk.eagle:library:535" package="TACTILE_SWITCH_PTH_RIGHT_ANGLE_KIT" package3d_urn="urn:adsk.eagle:package:40168/1" value="MOMENTARY-SWITCH-SPST-PTH-RIGHT-ANGLE-KIT" x="3" y="43" smashed="yes" rot="R270">
+<element name="BTN_SWITCH" library="SparkFun-Switches" library_urn="urn:adsk.eagle:library:535" package="TACTILE_SWITCH_PTH_RIGHT_ANGLE_KIT" package3d_urn="urn:adsk.eagle:package:40168/1" value="MOMENTARY-SWITCH-SPST-PTH-RIGHT-ANGLE-KIT" x="3" y="43" smashed="yes" rot="R270">
 <attribute name="NAME" x="1.286" y="43" size="0.6096" layer="25" font="vector" ratio="20" rot="R270" align="bottom-center"/>
 <attribute name="PROD_ID" value="CONN-10672" x="3" y="43" size="1.778" layer="27" rot="R270" display="off"/>
 <attribute name="SF_SKU" value="COM-10791" x="3" y="43" size="1.778" layer="27" rot="R270" display="off"/>
 </element>
-<element name="CHANGE_WEAPON" library="SparkFun-Switches" library_urn="urn:adsk.eagle:library:535" package="TACTILE_SWITCH_PTH_RIGHT_ANGLE_KIT" package3d_urn="urn:adsk.eagle:package:40168/1" value="MOMENTARY-SWITCH-SPST-PTH-RIGHT-ANGLE-KIT" x="3" y="33" smashed="yes" rot="R270">
+<element name="BTN_PISTE" library="SparkFun-Switches" library_urn="urn:adsk.eagle:library:535" package="TACTILE_SWITCH_PTH_RIGHT_ANGLE_KIT" package3d_urn="urn:adsk.eagle:package:40168/1" value="MOMENTARY-SWITCH-SPST-PTH-RIGHT-ANGLE-KIT" x="3" y="33" smashed="yes" rot="R270">
 <attribute name="NAME" x="1.286" y="33" size="0.6096" layer="25" font="vector" ratio="20" rot="R270" align="bottom-center"/>
 <attribute name="PROD_ID" value="CONN-10672" x="3" y="38" size="1.778" layer="27" rot="R270" display="off"/>
 <attribute name="SF_SKU" value="COM-10791" x="3" y="38" size="1.778" layer="27" rot="R270" display="off"/>
 </element>
-<element name="SWITCH_PLAYERS" library="SparkFun-Switches" library_urn="urn:adsk.eagle:library:535" package="TACTILE_SWITCH_PTH_RIGHT_ANGLE_KIT" package3d_urn="urn:adsk.eagle:package:40168/1" value="MOMENTARY-SWITCH-SPST-PTH-RIGHT-ANGLE-KIT" x="3" y="23" smashed="yes" rot="R270">
+<element name="BTN_CHANGE_WP" library="SparkFun-Switches" library_urn="urn:adsk.eagle:library:535" package="TACTILE_SWITCH_PTH_RIGHT_ANGLE_KIT" package3d_urn="urn:adsk.eagle:package:40168/1" value="MOMENTARY-SWITCH-SPST-PTH-RIGHT-ANGLE-KIT" x="3" y="23" smashed="yes" rot="R270">
 <attribute name="NAME" x="1.286" y="23" size="0.6096" layer="25" font="vector" ratio="20" rot="R270" align="bottom-center"/>
 <attribute name="PROD_ID" value="CONN-10672" x="3" y="28" size="1.778" layer="27" rot="R270" display="off"/>
@@
 <contactref element="NP_GND" pad="1"/>
 <polygon width="0.1524" layer="16">
-<vertex x="0" y="0"/>
-<vertex x="0" y="52"/>
-<vertex x="44" y="52"/>
-<vertex x="44" y="0"/>
+<vertex x="42" y="0"/>
+<vertex x="2" y="0" curve="-90"/>
+<vertex x="0" y="2"/>
+<vertex x="0" y="50" curve="-90"/>
+<vertex x="2" y="52"/>
+<vertex x="42" y="52" curve="-90"/>
+<vertex x="44" y="50"/>
+<vertex x="44" y="2" curve="-90"/>
 </polygon>
 <polygon width="0.1524" layer="1">
-<vertex x="0" y="0"/>
-<vertex x="0" y="52"/>
-<vertex x="44" y="52"/>
-<vertex x="44" y="0"/>
+<vertex x="42" y="0"/>
+<vertex x="2" y="0" curve="-90"/>
+<vertex x="0" y="2"/>
+<vertex x="0" y="50" curve="-90"/>
+<vertex x="2" y="52"/>
+<vertex x="42" y="52" curve="-90"/>
+<vertex x="44" y="50"/>
+<vertex x="44" y="2" curve="-90"/>
 </polygon>
 <contactref element="M1" pad="J1.4"/>
 <contactref element="M1" pad="J2.2"/>
 <contactref element="M2" pad="1"/>
-<contactref element="POT_5K" pad="2"/>
-<contactref element="CHANGE_WEAPON" pad="2"/>
-<contactref element="BTN_PISTE_MODE" pad="2"/>
-<contactref element="SWITCH_PLAYERS" pad="2"/>
+<contactref element="BTN_PISTE" pad="2"/>
+<contactref element="BTN_SWITCH" pad="2"/>
+<contactref element="BTN_CHANGE_WP" pad="2"/>
 <via x="32" y="41" extent="1-16" drill="0.35"/>
 <via x="15" y="20" extent="1-16" drill="0.35"/>
 <via x="33" y="16" extent="1-16" drill="0.35"/>
+<contactref element="BZR_GND" pad="1"/>
+<contactref element="POT_5K" pad="1"/>
 </signal>
 <signal name="5V">
@@
 <wire x1="20.15" y1="29.8687125" x2="20.15" y2="29.16" width="0.1524" layer="1"/>
 <wire x1="19.1674" y1="30.8513125" x2="20.15" y2="29.8687125" width="0.1524" layer="1"/>
+<contactref element="POT_5K" pad="3"/>
+<wire x1="13" y1="38" x2="16" y2="35" width="0.1524" layer="1"/>
+<wire x1="16" y1="35" x2="22" y2="35" width="0.1524" layer="1"/>
+<wire x1="22" y1="35" x2="22" y2="31.01" width="0.1524" layer="1"/>
+<wire x1="22" y1="31.01" x2="20.15" y2="29.16" width="0.1524" layer="1"/>
 </signal>
 <signal name="NEOPIXEL_DIN">
@@
 <wire x1="24.5" y1="13.5" x2="24.38" y2="13.3" width="0.1524" layer="1"/>
 </signal>
-<signal name="N$1">
-<contactref element="BZR_GND" pad="1"/>
-<contactref element="POT_5K" pad="3"/>
-<wire x1="21" y1="49" x2="13" y2="41" width="0.1524" layer="1"/>
-<wire x1="21" y1="49" x2="21" y2="50" width="0.1524" layer="1"/>
-<wire x1="13" y1="38" x2="13" y2="41" width="0.1524" layer="1"/>
-</signal>
-<signal name="PIN_BTN_PISTE_MODE">
-<contactref element="BTN_PISTE_MODE" pad="1"/>
+<signal name="PIN_BTN_SWITCH_SIDE">
+<contactref element="BTN_SWITCH" pad="1"/>
 <contactref element="M1" pad="J1.7"/>
 <wire x1="22" y1="31" x2="24" y2="29" width="0.1524" layer="16"/>
@@
 <wire x1="24" y1="29" x2="24.38" y2="28.54" width="0.1524" layer="16"/>
 </signal>
-<signal name="PIN_BTN_CHANGE_WEAPON">
-<contactref element="CHANGE_WEAPON" pad="1"/>
+<signal name="PIN_BTN_PISTE_MODE">
+<contactref element="BTN_PISTE" pad="1"/>
 <contactref element="M1" pad="J1.8"/>
 <wire x1="12.5" y1="26" x2="24.38" y2="26" width="0.1524" layer="16"/>
 <wire x1="3" y1="35.5" x2="12.5" y2="26" width="0.1524" layer="16"/>
 </signal>
-<signal name="PIN_BTN_SWITCH_PLAYERS">
-<contactref element="SWITCH_PLAYERS" pad="1"/>
+<signal name="PIN_BTN_CHANGE_WEAPON">
+<contactref element="BTN_CHANGE_WP" pad="1"/>
 <contactref element="M1" pad="J1.9"/>
 <wire x1="23" y1="24.5" x2="24" y2="23.5" width="0.1524" layer="16"/>
@@
 <wire x1="24" y1="23.5" x2="24.38" y2="23.46" width="0.1524" layer="16"/>
 </signal>
+<signal name="POT_IN">
+<contactref element="M1" pad="J2.9"/>
+<contactref element="POT_5K" pad="2"/>
+<wire x1="13" y1="43" x2="20.08" y2="43" width="0.1524" layer="16"/>
+<wire x1="24.78700625" y1="39.6826" x2="25.3626" y2="39.10700625" width="0.1524" layer="16"/>
+<wire x1="20.08" y1="43" x2="23.3974" y2="39.6826" width="0.1524" layer="16"/>
+<wire x1="25.3626" y1="37.7174" x2="39.62" y2="23.46" width="0.1524" layer="16"/>
+<wire x1="23.3974" y1="39.6826" x2="24.78700625" y2="39.6826" width="0.1524" layer="16"/>
+<wire x1="25.3626" y1="39.10700625" x2="25.3626" y2="37.7174" width="0.1524" layer="16"/>
+</signal>
 </signals>
